File: SlidersOfSociety-PCB.kicad_sch (KiCad schematic)
At the start: 21 parts, among them J1 Screw_Terminal_01x02, J2 6P4C, J3 6P4C, J4 Conn_01x06_Pin, J5 Conn_01x08_Pin, SW1 210-4MS, SW2 limit switch, U1 PIC18F25K83-I/SO, U2 DRV8871DDA, U3 MCP2561-E-SN

Commit message: idk what changed here, been some time
Parts:
- C1, C2: MANUFACTURER_PART_NUMBER CL21B105KBFNNNE -> (none); MPN (none) -> CL21B105KBFNNNE
- C3, C4: MANUFACTURER_PART_NUMBER CC0805KRX7R9BB104 -> (none); MPN (none) -> CC0805KRX7R9BB104
- C5: MANUFACTURER_PART_NUMBER UHE2A470MPD -> (none); MPN (none) -> UHE2A470MPD
- D1: MPN (none) -> 151031VS06000
- J1, SW2: now not fitted
- J2, J3: MANUFACTURER_PART_NUMBER MTJ-642BX2 -> (none); MPN (none) -> MTJ-642BX2
- R1, R4, R5: MANUFACTURER_PART_NUMBER CRCW080510K0FKEA -> (none); MPN (none) -> CRCW080510K0FKEA
- R2: MANUFACTURER_PART_NUMBER RC0805FR-07100RL -> (none); MPN (none) -> RC0805FR-07100RL
- R3: MANUFACTURER_PART_NUMBER RC0805FR-0756KL -> (none); MPN (none) -> RC0805FR-0756KL
- SW1: MANUFACTURER_PART_NUMBER 219-4MST -> (none); MPN (none) -> 219-4MST
- U1: MANUFACTURER_PART_NUMBER PIC18F25K83-I/SO -> (none); MPN (none) -> PIC18F25K83-I/SO
- U2: MANUFACTURER_PART_NUMBER DRV8871DDAR -> (none); MPN (none) -> DRV8871DDAR
- U3: MANUFACTURER_PART_NUMBER MCP2561T-E/SN -> (none); MPN (none) -> MCP2561T-E/SN
Connections:
- net at SW2.1 (A): now also U1.10 (OSC2_CLKOUT/RA6); no longer U1.12 (RC1/SOSCI)
- no-connect marks 12 -> 11
Changed lines of the file:
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@@
 	)
 	(no_connect
-		(at 105.41 130.81)
-	)
-	(no_connect
 		(at 135.89 115.57)
 	)
@@
 	(wire
 		(pts
+			(xy 92.71 144.78) (xy 92.71 148.59)
+		)
+		(stroke
+			(width 0)
+			(type default)
+		)
+	)
+	(wire
+		(pts
 			(xy 210.82 83.82) (xy 214.63 83.82)
 		)
@@
 	(wire
 		(pts
-			(xy 165.1 120.65) (xy 165.1 118.11)
+			(xy 177.8 91.44) (xy 177.8 92.71)
 		)
 		(stroke
@@
 	(wire
 		(pts
-			(xy 177.8 91.44) (xy 177.8 92.71)
+			(xy 107.95 30.48) (xy 107.95 36.83)
 		)
 		(stroke
@@
 	(wire
 		(pts
-			(xy 107.95 30.48) (xy 107.95 36.83)
+			(xy 92.71 130.81) (xy 105.41 130.81)
 		)
 		(stroke
@@
 	(wire
 		(pts
-			(xy 105.41 118.11) (xy 78.74 118.11)
+			(xy 92.71 134.62) (xy 92.71 130.81)
 		)
 		(stroke
@@
 	(wire
 		(pts
-			(xy 83.82 123.19) (xy 83.82 134.62)
+			(xy 105.41 118.11) (xy 78.74 118.11)
 		)
 		(stroke
@@
 	(wire
 		(pts
-			(xy 81.28 132.08) (xy 73.66 132.08)
+			(xy 83.82 123.19) (xy 83.82 134.62)
 		)
 		(stroke
@@
 	(wire
 		(pts
-			(xy 167.64 59.69) (xy 167.64 60.96)
+			(xy 81.28 132.08) (xy 73.66 132.08)
 		)
 		(stroke
@@
 	(wire
 		(pts
-			(xy 148.59 69.85) (xy 148.59 102.87)
+			(xy 167.64 59.69) (xy 167.64 60.96)
 		)
 		(stroke
@@
 	(wire
 		(pts
-			(xy 185.42 140.97) (xy 208.28 140.97)
+			(xy 148.59 69.85) (xy 148.59 102.87)
 		)
 		(stroke
@@
 	(wire
 		(pts
-			(xy 104.14 39.37) (xy 107.95 39.37)
+			(xy 185.42 140.97) (xy 208.28 140.97)
 		)
 		(stroke
@@
 	(wire
 		(pts
-			(xy 135.89 118.11) (xy 149.86 118.11)
+			(xy 104.14 39.37) (xy 107.95 39.37)
 		)
 		(stroke
@@
 	(wire
 		(pts
-			(xy 165.1 118.11) (xy 160.02 118.11)
-		)
-		(stroke
-			(width 0)
-			(type default)
-		)
-	)
-	(wire
-		(pts
 			(xy 214.63 63.5) (xy 210.82 63.5)
 		)
@@
 			)
 		)
-		(property "MANUFACTURER_PART_NUMBER" "CL21B105KBFNNNE"
+		(property "MPN" "CL21B105KBFNNNE"
 			(at 107.95 78.74 0)
 			(effects
@@
 	(symbol
 		(lib_id "Switch:SW_Push_Open")
-		(at 154.94 118.11 0)
+		(at 92.71 139.7 270)
 		(unit 1)
 		(exclude_from_sim no)
 		(in_bom yes)
 		(on_board yes)
-		(dnp no)
+		(dnp yes)
 		(fields_autoplaced yes)
 		(property "Reference" "SW2"
-			(at 154.94 111.76 0)
+			(at 95.25 138.4299 90)
 			(effects
 				(font
 					(size 1.27 1.27)
 				)
+				(justify left)
 			)
 		)
 		(property "Value" "limit switch"
-			(at 154.94 114.3 0)
+			(at 95.25 140.9699 90)
 			(effects
 				(font
 					(size 1.27 1.27)
 				)
+				(justify left)
 			)
 		)
 		(property "Footprint" "Connector_JST:JST_XH_B2B-XH-A_1x02_P2.50mm_Vertical"
-			(at 154.94 113.03 0)
+			(at 97.79 139.7 0)
 			(effects
 				(font
@@
 		)
 		(property "Datasheet" "~"
-			(at 154.94 113.03 0)
+			(at 97.79 139.7 0)
 			(effects
 				(font
@@
 		)
 		(property "Description" ""
-			(at 154.94 118.11 0)
-			(effects
-				(font
-					(size 1.27 1.27)
-				)
-			)
-		)
-		(property "MANUFACTURER_PART_NUMBER" ""
-			(at 154.94 118.11 0)
+			(at 92.71 139.7 0)
 			(effects
 				(font
 					(size 1.27 1.27)
 				)
-				(hide yes)
 			)
 		)
@@
 			)
 		)
-		(property "MANUFACTURER_PART_NUMBER" "CL21B105KBFNNNE"
+		(property "MPN" "CL21B105KBFNNNE"
 			(at 90.17 104.14 0)
 			(effects
@@
 			)
 		)
-		(property "MANUFACTURER_PART_NUMBER" "DRV8871DDAR"
+		(property "MPN" "DRV8871DDAR"
 			(at 175.26 140.97 0)
 			(effects
@@
 			)
 		)
-		(property "MANUFACTURER_PART_NUMBER" "CRCW080510K0FKEA"
+		(property "MPN" "CRCW080510K0FKEA"
 			(at 142.24 137.16 90)
 			(effects
@@
 			)
 		)
-		(property "MANUFACTURER_PART_NUMBER" ""
-			(at 63.5 105.41 0)
-			(effects
-				(font
-					(size 1.27 1.27)
-				)
-				(hide yes)
-			)
-		)
 		(pin "6"
 		)
@@
 			)
 		)
-		(property "MANUFACTURER_PART_NUMBER" "MCP2561T-E/SN"
+		(property "MPN" "MCP2561T-E/SN"
 			(at 177.8 74.93 0)
 			(effects
@@
 			)
 		)
-		(property "MANUFACTURER_PART_NUMBER" "CC0805KRX7R9BB104"
+		(property "MPN" "CC0805KRX7R9BB104"
 			(at 167.64 55.88 0)
 			(effects
@@
 			)
 		)
-		(property "MANUFACTURER_PART_NUMBER" ""
+		(property "MPN" "151031VS06000"
 			(at 142.24 148.59 90)
 			(effects
@@
 		(in_bom yes)
 		(on_board yes)
-		(dnp no)
+		(dnp yes)
 		(property "Reference" "J1"
 			(at 96.52 36.8299 0)
@@
 			)
 		)
-		(property "MANUFACTURER_PART_NUMBER" "CRCW080510K0FKEA"
+		(property "MPN" "CRCW080510K0FKEA"
 			(at 162.56 86.36 0)
 			(effects
@@
 			)
 		)
-		(property "MANUFACTURER_PART_NUMBER" "MTJ-642BX2"
+		(property "MPN" "MTJ-642BX2"
 			(at 224.79 86.36 0)
 			(effects
@@
 			)
 		)
-		(property "MANUFACTURER_PART_NUMBER" "RC0805FR-0756KL"
+		(property "MPN" "RC0805FR-0756KL"
 			(at 187.96 151.13 0)
 			(effects
@@
 	(symbol
 		(lib_id "power:GND")
-		(at 165.1 120.65 0)
+		(at 92.71 148.59 0)
 		(unit 1)
 		(exclude_from_sim no)
@@
 		(fields_autoplaced yes)
 		(property "Reference" "#PWR011"
-			(at 165.1 127 0)
+			(at 92.71 154.94 0)
 			(effects
 				(font
@@
 		)
 		(property "Value" "GND"
-			(at 165.1 125.73 0)
+			(at 92.71 153.67 0)
 			(effects
 				(font
@@
 		)
 		(property "Footprint" ""
-			(at 165.1 120.65 0)
+			(at 92.71 148.59 0)
 			(effects
 				(font
@@
 		)
 		(property "Datasheet" ""
-			(at 165.1 120.65 0)
+			(at 92.71 148.59 0)
 			(effects
 				(font
@@
 		)
 		(property "Description" "Power symbol creates a global label with name \"GND\" , ground"
-			(at 165.1 120.65 0)
+			(at 92.71 148.59 0)
 			(effects
 				(font
@@
 			)
 		)
-		(property "MANUFACTURER_PART_NUMBER" "PIC18F25K83-I/SO"
+		(property "MPN" "PIC18F25K83-I/SO"
 			(at 120.65 115.57 0)
 			(effects
@@
 			)
 		)
-		(property "MANUFACTURER_PART_NUMBER" "RC0805FR-07100RL"
+		(property "MPN" "RC0805FR-07100RL"
 			(at 97.79 97.79 90)
 			(effects
@@
 			)
 		)
-		(property "MANUFACTURER_PART_NUMBER" "MTJ-642BX2"
+		(property "MPN" "MTJ-642BX2"
 			(at 224.79 58.42 0)
 			(effects
@@
 			)
 		)
-		(property "MANUFACTURER_PART_NUMBER" ""
-			(at 213.36 133.35 0)
-			(effects
-				(font
-					(size 1.27 1.27)
-				)
-				(hide yes)
-			)
-		)
 		(pin "2"
 		)
@@
 			)
 		)
-		(property "MANUFACTURER_PART_NUMBER" "CC0805KRX7R9BB104"
+		(property "MPN" "CC0805KRX7R9BB104"
 			(at 180.34 121.92 0)
 			(effects
@@
 			)
 		)
-		(property "MANUFACTURER_PART_NUMBER" "CRCW080510K0FKEA"
+		(property "MPN" "CRCW080510K0FKEA"
 			(at 90.17 88.9 0)
 			(effects
@@
 			)
 		)
-		(property "MANUFACTURER_PART_NUMBER" "UHE2A470MPD"
+		(property "MPN" "UHE2A470MPD"
 			(at 193.04 121.92 0)
 			(effects
@@
 			)
 		)
-		(property "MANUFACTURER_PART_NUMBER" "219-4MST"
+		(property "MPN" "219-4MST"
 			(at 66.04 132.08 0)
 			(effects
